Commit message: Colorize gripper

File: ur10_robotiq_2f_140_description/urdf/robotiq_arg2f.xacro (robot description, xacro)
@@ -24,4 +24,7 @@
       </collision>
     </link>
+    <gazebo reference="${prefix}robotiq_arg2f_base_link">
+      <material>Gazebo/FlatBlack</material>
+    </gazebo>
   </xacro:macro>
   <xacro:macro name="finger_joints" params="prefix fingerprefix reflect">

File: ur10_robotiq_2f_140_description/urdf/robotiq_arg2f_140_model_macro.xacro (robot description, xacro)
@@ -31,4 +31,7 @@
       </collision>
     </link>
+    <gazebo reference="${prefix}${fingerprefix}_outer_knuckle">
+      <material>Gazebo/FlatBlack</material>
+    </gazebo>
   </xacro:macro>
   <xacro:macro name="outer_finger" params="prefix fingerprefix stroke">
@@ -61,4 +64,7 @@
       </collision>
     </link>
+    <gazebo reference="${prefix}${fingerprefix}_outer_finger">
+      <material>Gazebo/FlatBlack</material>
+    </gazebo>
   </xacro:macro>
   <xacro:macro name="inner_knuckle" params="prefix fingerprefix stroke">
@@ -91,4 +97,7 @@
       </collision>
     </link>
+    <gazebo reference="${prefix}${fingerprefix}_inner_knuckle">
+      <material>Gazebo/FlatBlack</material>
+    </gazebo>
   </xacro:macro>
   <xacro:macro name="inner_finger" params="prefix fingerprefix stroke">
@@ -121,4 +130,7 @@
       </collision>
     </link>
+    <gazebo reference="${prefix}${fingerprefix}_inner_finger">
+      <material>Gazebo/White</material>
+    </gazebo>
   </xacro:macro>
   <!-- Finger pad link, the default are the "big pads" with rubber-->
@@ -153,5 +165,5 @@
     </link>
     <gazebo reference="${prefix}${fingerprefix}_inner_finger_pad">
-      <selfCollide>true</selfCollide>
+      <material>Gazebo/White</material>
     </gazebo>
   </xacro:macro>

File: ur10_robotiq_2f_140_description/urdf/ur10_robotiq_2f_140_robot.urdf.xacro (robot description, xacro)
@@ -3,11 +3,11 @@
 	   name="ur10_robotiq_2f_140">
     <!-- Specifies simulated hardware interface used by gazebo.
-				 Although the real hardware uses a position joint interface, it makes more sense to
-				 use the 'EffortJointInterface' for simulation.
-				 This is because when using the 'PositionJointInterface', gazebo uses
-				 the Joint.SetPosition() method which forces the simulation to adapt the specified joint
-				 position and may lead to weird behaviors in collisions.
-				 Note that, when using the 'EffortJointInterface', you also have to specify
-				 a 'effort_controllers/JointTrajectoryController' controller which requires to set PID gains.
+		 Although the real hardware uses a position joint interface, it makes more sense to
+		 use the 'EffortJointInterface' for simulation.
+		 This is because when using the 'PositionJointInterface', gazebo uses
+		 the Joint.SetPosition() method which forces the simulation to adapt the specified joint
+		 position and may lead to weird behaviors in collisions.
+		 Note that, when using the 'EffortJointInterface', you also have to specify
+		a 'effort_controllers/JointTrajectoryController' controller which requires to set PID gains.
      -->
     <xacro:arg name="arm_transmission_hw_interface" default="hardware_interface/PositionJointInterface"/>
@@ -18,10 +18,10 @@
     <xacro:arg name="limited" default="false"/>
 	<xacro:include filename="$(find ur10_robotiq_2f_140_description)/urdf/ur10_robotiq_2f_140.urdf.xacro" />
-	<!-- Universal robot UR10 with Robotiq 2f 140 gripper -->
+	<!-- universal robot UR10 with Robotiq 2f 140 gripper -->
 	<xacro:ur10_robotiq_2f_140_robot prefix="" joint_limited="$(arg limited)"
 		arm_transmission_hw_interface="$(arg arm_transmission_hw_interface)"
 		gripper_transmission_hw_interface="$(arg gripper_transmission_hw_interface)"
 	/>
-	<!-- world frame -->
+	<!-- used for fixing robot to Gazebo 'base_link' -->
 	<link name="world" />
 	<!-- attach ur10 to world frame -->
