Commit message: Generate movit package

File: ur10_robotiq_2f_140_description/urdf/ur10_robotiq_2f_140.urdf.xacro (robot description, xacro)
@@ -29,5 +29,5 @@
       <parent link="${prefix}tool0"/>
       <child link="${prefix}robotiq_arg2f_base_link"/>
-      <origin xyz="0 0 0.001" rpy="0 0 ${pi/2}"/>
+      <origin xyz="0 0 0" rpy="0 0 ${pi/2}"/>
     </joint>
   </xacro:macro>
