Commit message: Add tf_prefix as argument in spawn.launch

File: ur10_robotiq_2f_140_description/urdf/ur10_robotiq_2f_140_robot.urdf.xacro (robot description, xacro)
@@ -29,5 +29,5 @@
 		<parent link="world" />
 		<child link = "base_link" />
-		<origin xyz="0 0 0.3" rpy="0 0 0" />
+		<origin xyz="0 0 0" rpy="0 0 0" />
 	</joint>
 	<!-- load ros_control gazebo plugin -->
