Commit message: dark grey as knuckle color

File: ur10_robotiq_2f_140_description/urdf/robotiq_arg2f_140_model_macro.xacro (robot description, xacro)
@@ -32,5 +32,5 @@
     </link>
     <gazebo reference="${prefix}${fingerprefix}_outer_knuckle">
-      <material>Gazebo/FlatBlack</material>
+      <material>Gazebo/DarkGrey</material>
     </gazebo>
   </xacro:macro>
@@ -131,5 +131,5 @@
     </link>
     <gazebo reference="${prefix}${fingerprefix}_inner_finger">
-      <material>Gazebo/White</material>
+      <material>Gazebo/DarkGrey</material>
     </gazebo>
   </xacro:macro>
@@ -165,5 +165,5 @@
     </link>
     <gazebo reference="${prefix}${fingerprefix}_inner_finger_pad">
-      <material>Gazebo/White</material>
+      <material>Gazebo/DarkGrey</material>
     </gazebo>
   </xacro:macro>

Commit message: Pass world pose in xacro

File: ur10_robotiq_2f_140_description/urdf/robotiq_arg2f_140_model_macro.xacro (robot description, xacro)
@@ -165,4 +165,27 @@
     </link>
     <gazebo reference="${prefix}${fingerprefix}_inner_finger_pad">
+      <collision name="${prefix}${fingerprefix}_inner_finger_pad">
+        <surface>
+          <friction>
+            <torsional>
+              <coefficient>10.0</coefficient>
+              <use_patch_radius>true</use_patch_radius>
+              <patch_radius>0.05</patch_radius>
+            </torsional>
+          </friction>
+          <contact>
+            <poissons_ratio>0.5</poissons_ratio>
+            <elastic_modulus>1e8</elastic_modulus>
+          </contact>
+        </surface>
+      </collision>
+      <mu1>10</mu1>
+      <mu2>10</mu2>
+      <maxVel>1</maxVel>
+      <kp>1000000.0</kp>
+      <kd>100.0</kd>
+      <fdir1>0 0 1</fdir1>
+      <minDepth>0.0</minDepth>
+      <maxContacts>100</maxContacts>
       <material>Gazebo/DarkGrey</material>
     </gazebo>

File: ur10_robotiq_2f_140_description/urdf/ur10_robotiq_2f_140.urdf.xacro (robot description, xacro)
@@ -31,4 +31,22 @@
       <origin xyz="0 0 0" rpy="0 0 ${pi/2}"/>
     </joint>
+    <!-- grasp plugin for fixing unstable grasping physics -->
+    <gazebo>
+      <plugin name="gazebo_grasp_fix" filename="libgazebo_grasp_fix.so">
+        <arm>
+          <arm_name>ur10-arm</arm_name>
+          <palm_link>${prefix}wrist_3_link</palm_link>
+          <gripper_link>${prefix}left_inner_finger</gripper_link>
+          <gripper_link>${prefix}right_inner_finger</gripper_link>
+        </arm>
+        <forces_angle_tolerance>100</forces_angle_tolerance>
+        <update_rate>4</update_rate>
+        <grip_count_threshold>4</grip_count_threshold>
+        <max_grip_count>8</max_grip_count>
+        <release_tolerance>0.005</release_tolerance>
+        <disable_collisions_on_attach>false</disable_collisions_on_attach>
+        <contact_topic>__default_topic__</contact_topic>
+      </plugin>
+    </gazebo>
   </xacro:macro>
 </robot>

File: ur10_robotiq_2f_140_description/urdf/ur10_robotiq_2f_140_robot.urdf.xacro (robot description, xacro)
@@ -17,4 +17,11 @@
     -->
     <xacro:arg name="limited" default="false"/>
+	<!-- position and rotation of the robot in the world frame -->
+	<xacro:arg name="x" default="0.0"/>
+	<xacro:arg name="y" default="0.0"/>
+	<xacro:arg name="z" default="0.0"/>
+	<xacro:arg name="roll" default="0.0"/>
+	<xacro:arg name="pitch" default="0.0"/>
+	<xacro:arg name="yaw" default="0.0"/>
 	<xacro:include filename="$(find ur10_robotiq_2f_140_description)/urdf/ur10_robotiq_2f_140.urdf.xacro" />
 	<!-- universal robot UR10 with Robotiq 2f 140 gripper -->
@@ -29,5 +36,5 @@
 		<parent link="world" />
 		<child link = "base_link" />
-		<origin xyz="0 0 0" rpy="0 0 0" />
+		<origin xyz="$(arg x) $(arg y) $(arg z)" rpy="$(arg roll) $(arg pitch) $(arg yaw)" />
 	</joint>
 	<!-- load ros_control gazebo plugin -->

Commit message: Make gripper control left and right joints separately

File: ur10_robotiq_2f_140_description/urdf/robotiq_arg2f_140_model_macro.xacro (robot description, xacro)
@@ -206,5 +206,5 @@
       <axis xyz="1 0 0" />
       <limit lower="-0.8757" upper="0.8757" velocity="2.0" effort="1000" />
-      <mimic joint="${prefix}finger_joint" multiplier="-1" offset="0" />
+      <mimic joint="${prefix}${fingerprefix}_finger_joint" multiplier="-1" offset="0" />
     </joint>
   </xacro:macro>
@@ -216,5 +216,5 @@
       <axis xyz="1 0 0" />
       <limit lower="-0.8757" upper="0.8757" velocity="2.0" effort="1000" />
-      <mimic joint="${prefix}finger_joint" multiplier="1" offset="0" />
+      <mimic joint="${prefix}${fingerprefix}_finger_joint" multiplier="1" offset="0" />
     </joint>
   </xacro:macro>
@@ -228,6 +228,6 @@
   </xacro:macro>
   <xacro:include filename="$(find ur10_robotiq_2f_140_description)/urdf/robotiq_arg2f.xacro" />
-  <xacro:macro name="finger_joint" params="prefix">
-    <joint name="${prefix}finger_joint" type="revolute">
+  <xacro:macro name="left_finger" params="prefix">
+    <joint name="${prefix}left_finger_joint" type="revolute">
       <origin xyz="0 -0.030601 0.054905" rpy="${pi / 2 + .725} 0 0" />
       <parent link="${prefix}robotiq_arg2f_base_link" />
@@ -237,22 +237,21 @@
     </joint>
     <xacro:finger_joints prefix="${prefix}" fingerprefix="left" reflect="1.0"/>
-  </xacro:macro>
-  <xacro:macro name="right_outer_knuckle_joint" params="prefix">
-    <joint name="${prefix}right_outer_knuckle_joint" type="revolute">
+    <xacro:finger_links prefix="${prefix}" fingerprefix="left" stroke="140"/>
+  </xacro:macro>
+  <xacro:macro name="right_finger" params="prefix">
+    <joint name="${prefix}right_finger_joint" type="revolute">
       <origin xyz="0 0.030601 0.054905" rpy="${pi / 2 + .725} 0 ${pi}" />
       <parent link="${prefix}robotiq_arg2f_base_link" />
       <child link="${prefix}right_outer_knuckle" />
-      <axis xyz="1 0 0" />
-      <limit lower="-0.725" upper="0.725" velocity="2.0" effort="1000" />
-      <mimic joint="${prefix}finger_joint" multiplier="-1" offset="0" />
+      <axis xyz="-1 0 0" />
+      <limit lower="0" upper="0.7" velocity="2.0" effort="1000" />
     </joint>
     <xacro:finger_joints prefix="${prefix}" fingerprefix="right" reflect="-1.0"/>
+    <xacro:finger_links prefix="${prefix}" fingerprefix="right" stroke="140"/>
   </xacro:macro>
   <xacro:macro name="robotiq_arg2f_140" params="prefix transmission_hw_interface:=hardware_interface/PositionJointInterface">
     <xacro:robotiq_arg2f_base_link prefix="${prefix}"/>
-    <xacro:finger_links prefix="${prefix}" fingerprefix="left" stroke="140"/>
-    <xacro:finger_links prefix="${prefix}" fingerprefix="right" stroke="140"/>
-    <xacro:finger_joint prefix="${prefix}"/>
-    <xacro:right_outer_knuckle_joint prefix="${prefix}"/>
+    <xacro:left_finger prefix="${prefix}"/>
+    <xacro:right_finger prefix="${prefix}"/>
     <xacro:robotiq_arg2f_transmission prefix="${prefix}" hw_interface="${transmission_hw_interface}"/>
   </xacro:macro>

File: ur10_robotiq_2f_140_description/urdf/robotiq_arg2f_transmission.xacro (robot description, xacro)
@@ -2,10 +2,19 @@
 <robot xmlns:xacro="http://ros.org/wiki/xacro">
   <xacro:macro name="robotiq_arg2f_transmission" params="prefix hw_interface">
-    <transmission name="${prefix}finger_joint_trans">
+    <transmission name="${prefix}left_finger_joint_trans">
       <type>transmission_interface/SimpleTransmission</type>
-      <joint name="${prefix}finger_joint">
+      <joint name="${prefix}left_finger_joint">
         <hardwareInterface>${hw_interface}</hardwareInterface>
       </joint>
-      <actuator name="${prefix}finger_joint_motor">
+      <actuator name="${prefix}left_finger_joint_motor">
+        <mechanicalReduction>1</mechanicalReduction>
+      </actuator>
+    </transmission>
+    <transmission name="${prefix}right_finger_joint_trans">
+      <type>transmission_interface/SimpleTransmission</type>
+      <joint name="${prefix}right_finger_joint">
+        <hardwareInterface>${hw_interface}</hardwareInterface>
+      </joint>
+      <actuator name="${prefix}right_finger_joint_motor">
         <mechanicalReduction>1</mechanicalReduction>
       </actuator>
@@ -13,27 +22,13 @@
     <gazebo>
       <!-- loading plugin: mimic joints works in gazebo now-->
-      <plugin filename="libroboticsgroup_gazebo_mimic_joint_plugin.so" name="${prefix}mimic_robotiq_140_4">
-        <joint>${prefix}finger_joint</joint>
-        <mimicJoint>${prefix}right_outer_knuckle_joint</mimicJoint>
-        <multiplier>-1.0</multiplier>
-        <offset>0.0</offset>
-        <hasPID />
-      </plugin>
       <plugin filename="libroboticsgroup_gazebo_mimic_joint_plugin.so" name="${prefix}mimic_robotiq_140_2">
-        <joint>${prefix}finger_joint</joint>
+        <joint>${prefix}left_finger_joint</joint>
         <mimicJoint>${prefix}left_inner_finger_joint</mimicJoint>
         <multiplier>1.0</multiplier>
-        <offset>0.0</offset>
-        <hasPID />
-      </plugin>
-      <plugin filename="libroboticsgroup_gazebo_mimic_joint_plugin.so" name="${prefix}mimic_robotiq_140_1">
-        <joint>${prefix}finger_joint</joint>
-        <mimicJoint>${prefix}right_inner_finger_joint</mimicJoint>
-        <multiplier>1.0</multiplier>
-        <offset>0.0</offset>
+        <offset>-0.02</offset>
         <hasPID />
       </plugin>
       <plugin filename="libroboticsgroup_gazebo_mimic_joint_plugin.so" name="${prefix}mimic_robotiq_140_3">
-        <joint>${prefix}finger_joint</joint>
+        <joint>${prefix}left_finger_joint</joint>
         <mimicJoint>${prefix}left_inner_knuckle_joint</mimicJoint>
         <multiplier>-1.0</multiplier>
@@ -41,6 +36,13 @@
         <hasPID />
       </plugin>
+      <plugin filename="libroboticsgroup_gazebo_mimic_joint_plugin.so" name="${prefix}mimic_robotiq_140_1">
+        <joint>${prefix}right_finger_joint</joint>
+        <mimicJoint>${prefix}right_inner_finger_joint</mimicJoint>
+        <multiplier>1.0</multiplier>
+        <offset>-0.02</offset>
+        <hasPID />
+      </plugin>
       <plugin filename="libroboticsgroup_gazebo_mimic_joint_plugin.so" name="${prefix}mimic_robotiq_140_5">
-        <joint>${prefix}finger_joint</joint>
+        <joint>${prefix}right_finger_joint</joint>
         <mimicJoint>${prefix}right_inner_knuckle_joint</mimicJoint>
         <multiplier>-1.0</multiplier>

Commit message: Add tcp link to gripper

File: ur10_robotiq_2f_140_description/urdf/robotiq_arg2f_140_model_macro.xacro (robot description, xacro)
@@ -250,8 +250,17 @@
     <xacro:finger_links prefix="${prefix}" fingerprefix="right" stroke="140"/>
   </xacro:macro>
+  <xacro:macro name="tcp" params="prefix">
+    <link name="${prefix}tcp" />
+    <joint name="${prefix}tcp_joint" type="fixed">
+      <origin xyz="0 0 0.177" rpy="0 0 0" />
+      <parent link="${prefix}robotiq_arg2f_base_link" />
+      <child link="${prefix}tcp" />
+    </joint>
+  </xacro:macro>
   <xacro:macro name="robotiq_arg2f_140" params="prefix transmission_hw_interface:=hardware_interface/PositionJointInterface">
     <xacro:robotiq_arg2f_base_link prefix="${prefix}"/>
     <xacro:left_finger prefix="${prefix}"/>
     <xacro:right_finger prefix="${prefix}"/>
+    <xacro:tcp prefix="${prefix}"/>
     <xacro:robotiq_arg2f_transmission prefix="${prefix}" hw_interface="${transmission_hw_interface}"/>
   </xacro:macro>
